File: SimpleSerialCard.kicad_sch (KiCad schematic)
At the start: 17 parts, among them J1 IRQ ENABLE, J2 RS-232 OUT, P1 A2Bus, U1 74HCT245, U2 28C256, U3 1.8432M, U4 SSCGLU, U5 W65C51NxP, U6 MC1489, U7 MC1488

Commit message: reroute everything
Parts:
- added ALT_U3: 1.8432M, Oscillator:Oscillator_DIP-14, symbol Oscillator:TCXO-14
- added C10, C9: 0.01u, Capacitor_THT:C_Disc_D4.3mm_W1.9mm_P5.00mm, symbol Device:C_Small
- added C12, C13, C14: 330p, Capacitor_THT:C_Disc_D3.0mm_W1.6mm_P2.50mm, symbol Device:C_Small
- added C8: 0.1u, Capacitor_THT:C_Disc_D4.3mm_W1.9mm_P5.00mm, symbol Device:C_Small
- renumbered U7 to U6, U6 to U7
Connections:
- net +12V: now also P1.50 (+12V), C10.1, C8.1
- net +5V: now also ALT_U3.14 (Vcc); no longer C7.1
- net -12V: now also C7.2, P1.33 (-12V), C9.2
- net GND: now also C7.1, ALT_U3.7 (GND), C10.2, C12.2, C13.2, C14.2, C8.2, C9.1; no longer C7.2
- net SERCLK: now also ALT_U3.8 (OUT)
- net at U5.10 (TxD): now also U6.4 (IB1); no longer U6.9 (IC2)
- net at U5.11 (~{DTR}): now also U6.9 (IC2); no longer U6.12 (ID2)
- net at U5.12 (RxD): now also U7.6 (OB); no longer U7.3 (OA)
- net at U5.16 (~{DCD}): now also U7.3 (OA); no longer U7.6 (OB)
- net at U5.17 (~{DSR}): now also U7.8 (OC); no longer U7.11 (OD)
- net at U5.8 (~{RTS}): now also U6.12 (ID2); no longer U6.4 (IB1)
- net at U4.2 (CTS), U5.9 (~{CTS}): now also U7.11 (OD); no longer U7.8 (OC)
- net CTS: no longer names the net of U7.10 (IC)
- net CTS: now also J2.6 (DSR); no longer J2.8 (CTS)
- net DCD: no longer names the net of J2.1 (DCD)
- net DCD: now also U7.1 (IA); no longer U7.4 (IB)
- net DSR: no longer names the net of U7.13 (ID)
- net DSR: now also J2.8 (CTS); no longer J2.6 (DSR)
- net DTR: no longer names the net of J2.4 (DTR)
- net DTR: now also U6.8 (OC), C13.1; no longer U6.11 (OD)
- net RTS: no longer names the net of U6.6 (OB)
- net RTS: now also J2.3 (TxD), C12.1; no longer J2.7 (RTS)
- net RXD: no longer names the net of J2.2 (RxD)
- net RXD: now also U7.4 (IB); no longer U7.1 (IA)
- removed net TXD: J2.3 (TxD), U6.8 (OC)
- new net: C14.1, J2.7 (RTS), U6.11 (OD)
- no-connect marks 27 -> 25
Other:
- note added: "Omit capacitors for 14C88"
- moved on the sheet: U3
